File: Graduation_Cap.kicad_pcb (KiCad board)
At the start: 2 copper layers, 220 x 220 mm, 133 parts, among them J1 USB, Q1 PN2222A, Q2 PN2222A, Q3 PN2222A, Q4 PN2222A, Q5 PN2222A, Q6 PN2222A, Q7 PN2222A, Q8 PN2222A, U1 7805, U2 NE555P, U3 74HC595

Commit message: upd
Parts:
- renumbered D40 to D29, D41 to D30, D42 to D31, D43 to D32, D44 to D33, D45 to D34, D46 to D35, D47 to D36, D48 to D37, D49 to D38, D50 to D39, D51 to D40, D52 to D41, D53 to D42, D54 to D43, D55 to D44, D56 to D45, D57 to D46, D58 to D47, D59 to D48, D60 to D49, D61 to D50, D62 to D51, D63 to D52, D64 to D53, D65 to D54, D66 to D55, D67 to D56, D68 to D57, D69 to D58, D70 to D59, D71 to D60, D72 to D61, D73 to D62, D74 to D63, D75 to D64, D76 to D65, D77 to D66, D78 to D67, D79 to D68, D80 to D69, D81 to D70, D82 to D71, D83 to D72, D84 to D73, D85 to D74, D86 to D75, D87 to D76, D88 to D77, D89 to D78, D90 to D79, D91 to D80, Q3 to Q2, Q4 to Q3, Q5 to Q4, Q6 to Q5, Q7 to Q6, Q8 to Q7, R12 to R10, R13 to R11, R14 to R12, R15 to R13, R16 to R14, R17 to R15, R4 to R3, R5 to R4, R7 to R5, R8 to R6, R9 to R7, R10 to R8, R11 to R9
Connections:
- J1 pad 2: Net-(J1-Pad2) -> unconnected-(J1-D--Pad2)
- J1 pad 3: Net-(J1-Pad3) -> unconnected-(J1-D+-Pad3)
- J1 pad 4: Net-(J1-Pad4) -> unconnected-(J1-ID-Pad4)
- J1 pad 6: Net-(J1-Pad6) -> unconnected-(J1-Shield-Pad6)_0
- U2 pad 5: Net-(U2-Pad5) -> unconnected-(U2-CONT-Pad5)
- U2 pad 7: Net-(U2-Pad7) -> unconnected-(U2-DIS-Pad7)
- U3 pad 3: Net-(R6-Pad2) -> unconnected-(U3-Qd-Pad3)
- U3 pad 7: Net-(U3-Pad7) -> unconnected-(U3-Qh-Pad7)
Other:
- net class Default removed
